Commit message: turtlebot2 model updated

File: turtlebot2 simu docker/turtlebot2/turtlebot2/urdf/turtlebot2.urdf (robot description, URDF)
Before this commit: robot turtlebot2, 24 links, 23 joints
Links:
- link base_link: geometry collision cylinder length=0.10938 radius=0.178; visual mesh filename=/home/turtlebot2_ws/src/kobuki_description/meshes/main_body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
- link wheel_left_link: geometry collision cylinder length=0.0206 radius=0.035; visual mesh filename=/home/turtlebot2_ws/src/kobuki_description/meshes/wheel.dae
- link wheel_right_link: geometry collision cylinder length=0.0206 radius=0.035; visual mesh filename=/home/turtlebot2_ws/src/kobuki_description/meshes/wheel.dae
